Commit message: nemo-ws repos from robot

File: nemo/articubot_one/description/lidar.xacro (robot description, xacro)
@@ -4,5 +4,5 @@
         <parent link="base_link"/>
         <child link="base_scan"/>
-        <origin xyz="0.04 0 0.27" rpy="0 0 0"/>
+        <origin xyz="0 0 0.27" rpy="0 0 0"/>
     </joint>
     <link name="base_scan">

File: nemo/articubot_one/description/ros2_control.xacro (robot description, xacro)
@@ -7,7 +7,7 @@
                 <param name="left_wheel_name">left_wheel_joint</param>
                 <param name="right_wheel_name">right_wheel_joint</param>
-                <param name="loop_rate">100</param>
+                <param name="loop_rate">50</param>
                 <param name="device">/dev/ttyUSB0</param>
-                <param name="baud_rate">57600</param>
+                <param name="baud_rate">230400</param>
                 <param name="timeout">1000</param>
                 <param name="enc_counts_per_rev">92800</param>
